File: Keypad.kicad_pcb (KiCad board)
At the start: 2 copper layers, 109 x 57.2 mm, 46 parts, among them J1 10118193-0001LF, J2 M20-9750446, Q1 BC32725TA, SW1 MX1A-11NN, SW2 MX1A-11NN, SW3 MX1A-11NN, SW4 MX1A-11NN, SW5 MX1A-11NN, SW6 MX1A-11NN, SW7 MX1A-11NN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

Commit message: Upadated schematic
Changed lines of the file:
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@@
     (descr "TO-92 leads molded, narrow, drill 0.75mm (see NXP sot054_po.pdf)")
     (tags "to-92 sc-43 sc-43a sot54 PA33 transistor")
-    (fp_text reference Q1 (at -3.7592 0.0254) (layer F.SilkS)
-      (effects (font (size 1 1) (thickness 0.2)))
+    (fp_text reference Q1 (at -4.2672 0.0254) (layer F.SilkS)
+      (effects (font (size 1.5 1.5) (thickness 0.2)))
     )
     (fp_text value BC32725TA (at 0 -5.207) (layer F.Fab)
@@
     (tags capacitor)
     (attr smd)
-    (fp_text reference C5 (at -2.42824 0 180) (layer F.SilkS)
+    (fp_text reference C5 (at -0.01524 1.9558 180) (layer F.SilkS)
       (effects (font (size 1 1) (thickness 0.2)))
     )
@@
     (tags capacitor)
     (attr smd)
-    (fp_text reference C4 (at -0.00254 1.6764) (layer F.SilkS)
-      (effects (font (size 1 1) (thickness 0.2)))
-    )
+    (fp_text reference C4 (at -0.00254 -1.5748) (layer F.SilkS)
+      (effects (font (size 1 1) (thickness 0.2)))
+    )
